Commit message: Created hawaii gazebo package and updated urdf files

File: hawaii_ros_ws/src/hawaii_descriptions/urdf/hawaii.urdf.xacro (robot description, xacro)
@@ -1,17 +1,48 @@
 <?xml version="1.0"?>
 <robot name="hawaii" xmlns:xacro="http://ros.org/wiki/xacro">
-  <xacro:arg name="robot_name" default="hawaii"/>
-  <xacro:arg name="base_link_frame" default="base_link"/>
-  <xacro:arg name="show_ar_tag" default="false"/>
-  <xacro:arg name="show_gripper_bar" default="true"/>
-  <xacro:arg name="show_gripper_fingers" default="true"/>
-  <xacro:arg name="use_world_frame" default="true"/>
-  <xacro:arg name="external_urdf_loc" default=""/>
-  <xacro:arg name="load_gazebo_configs" default="false"/>
-  <xacro:property name="urdf_loc" value="$(arg external_urdf_loc)"/>
-  <xacro:property name="pi_offset" value="0.00001"/>
-  <xacro:if value="$(arg load_gazebo_configs)">
-    <xacro:include filename="$(find interbotix_xsarm_gazebo)/config/interbotix_texture.gazebo"/>
-  </xacro:if>
+  <xacro:property name="robot_model"
+    value="hawaii"
+    scope="global"/>
+  <xacro:property name="dof"
+    value="5"
+    scope="global"/>
+  <xacro:arg name="robot_name"                      default="${robot_model}"/>
+  <xacro:arg name="base_link_frame"                 default="base_link"/>
+  <xacro:arg name="use_gripper"                     default="true"/>
+  <xacro:arg name="show_ar_tag"                     default="false"/>
+  <xacro:arg name="show_gripper_bar"                default="true"/>
+  <xacro:arg name="show_gripper_fingers"            default="true"/>
+  <xacro:arg name="use_world_frame"                 default="false"/>
+  <xacro:arg name="external_urdf_loc"               default=""/>
+  <xacro:arg name="hardware_type"                   default="actual"/>
+  <xacro:property name="mesh_directory"             value="package://hawaii_descriptions/meshes"/>
+  <xacro:property name="urdf_loc"                   value="$(arg external_urdf_loc)"/>
+  <xacro:property name="hardware_type"              value="$(arg hardware_type)"/>
+  <xacro:property name="pi_offset"                  value="0.00001"/>
+  <xacro:property name="waist_limit_effort"         value="10"/>
+  <xacro:property name="waist_limit_lower"          value="${-pi + pi_offset}"/>
+  <xacro:property name="waist_limit_upper"          value="${pi - pi_offset}"/>
+  <xacro:property name="waist_limit_vel"            value="${pi}"/>
+  <xacro:property name="shoulder_limit_effort"      value="20"/>
+  <xacro:property name="shoulder_limit_lower"       value="${radians(-106)}"/>
+  <xacro:property name="shoulder_limit_upper"       value="${radians(72)}"/>
+  <xacro:property name="shoulder_limit_vel"         value="${pi}"/>
+  <xacro:property name="elbow_limit_effort"         value="15"/>
+  <xacro:property name="elbow_limit_lower"          value="${radians(-101)}"/>
+  <xacro:property name="elbow_limit_upper"          value="${radians(92)}"/>
+  <xacro:property name="elbow_limit_vel"            value="${pi}"/>
+  <xacro:property name="wrist_angle_limit_effort"   value="5"/>
+  <xacro:property name="wrist_angle_limit_lower"    value="${radians(-107)}"/>
+  <xacro:property name="wrist_angle_limit_upper"    value="${radians(128)}"/>
+  <xacro:property name="wrist_angle_limit_vel"      value="${pi}"/>
+  <xacro:property name="wrist_rotate_limit_effort"  value="1"/>
+  <xacro:property name="wrist_rotate_limit_lower"   value="${-pi + pi_offset}"/>
+  <xacro:property name="wrist_rotate_limit_upper"   value="${pi - pi_offset}"/>
+  <xacro:property name="wrist_rotate_limit_vel"     value="${pi}"/>
+  <xacro:property name="gripper_limit_vel"          value="${pi}"/>
+  <xacro:property name="finger_limit_effort"        value="5"/>
+  <xacro:property name="finger_limit_lower"         value="0.021"/>
+  <xacro:property name="finger_limit_upper"         value="0.057"/>
+  <xacro:property name="finger_limit_vel"           value="1"/>
   <material name="interbotix_black">
     <texture filename="package://hawaii_descriptions/meshes/interbotix_black.png"/>
@@ -20,423 +51,611 @@
     <link name="world"/>
     <joint name="fixed" type="fixed">
-      <parent link="world"/>
-      <child link="$(arg robot_name)/$(arg base_link_frame)"/>
+      <parent
+        link="world"/>
+      <child
+        link="$(arg robot_name)/$(arg base_link_frame)"/>
     </joint>
-  </xacro:if>
+  </xacro:if> <!-- use_world_frame -->
   <link name="$(arg robot_name)/$(arg base_link_frame)">
     <visual>
-      <origin rpy="0 0 ${pi/2}" xyz="0 0 0"/>
-      <geometry>
-        <mesh filename="package://hawaii_descriptions/meshes/vx300_1_base.stl" scale="0.001 0.001 0.001"/>
+      <origin
+        rpy="0 0 ${pi/2}"
+        xyz="0 0 0"/>
+      <geometry>
+        <mesh
+          filename="${mesh_directory}/base.stl"
+          scale="0.001 0.001 0.001"/>
       </geometry>
       <material name="interbotix_black"/>
     </visual>
     <collision>
-      <origin rpy="0 0 ${pi/2}" xyz="0 0 0"/>
-      <geometry>
-        <mesh filename="package://hawaii_descriptions/meshes/vx300_1_base.stl" scale="0.001 0.001 0.001"/>
+      <origin
+        rpy="0 0 ${pi/2}"
+        xyz="0 0 0"/>
+      <geometry>
+        <mesh
+          filename="${mesh_directory}/base.stl"
+          scale="0.001 0.001 0.001"/>
       </geometry>
     </collision>
     <inertial>
-      <origin rpy="0 0 ${pi/2}" xyz="-0.0534774000 -0.0005625750 0.0205961000"/>
-      <mass value="0.969034" />
-      <inertia ixx="0.0060240000" iyy="0.0017000000" izz="0.0071620000" ixy="0.0000471300" ixz="0.0000038510" iyz="-0.0000841500" />
+      <origin
+        rpy="0 0 ${pi/2}"
+        xyz="-0.0534774000 -0.0005625750 0.0205961000"/>
+      <mass value="0.969034"/>
+      <inertia
+        ixx="0.0060240000"
+        iyy="0.0017000000"
+        izz="0.0071620000"
+        ixy="0.0000471300"
+        ixz="0.0000038510"
+        iyz="-0.0000841500"/>
     </inertial>
   </link>
   <joint name="waist" type="revolute">
     <axis xyz="0 0 1"/>
-    <limit effort="10" lower="${-pi + pi_offset}" upper="${pi - pi_offset}" velocity="${pi}"/>
-    <origin rpy="0 0 0" xyz="0 0 0.079"/>
-    <parent link="$(arg robot_name)/$(arg base_link_frame)"/>
-    <child link="$(arg robot_name)/shoulder_link"/>
-    <dynamics friction="0.1"/>
+    <limit
+      effort="${waist_limit_effort}"
+      lower="${waist_limit_lower}"
+      upper="${waist_limit_upper}"
+      velocity="${waist_limit_vel}"/>
+    <origin
+      rpy="0 0 0"
+      xyz="0 0 0.079"/>
+    <parent
+      link="$(arg robot_name)/$(arg base_link_frame)"/>
+    <child
+      link="$(arg robot_name)/shoulder_link"/>
+    <dynamics
+      friction="0.1"
+      damping="0.1"/>
   </joint>
-  <transmission name="trans_waist">
-    <type>transmission_interface/SimpleTransmission</type>
-    <joint name="waist">
-      <hardwareInterface>hardware_interface/EffortJointInterface</hardwareInterface>
-    </joint>
-    <actuator name="waist_motor">
-      <mechanicalReduction>1</mechanicalReduction>
-    </actuator>
-  </transmission>
   <link name="$(arg robot_name)/shoulder_link">
     <visual>
-      <origin rpy="0 0 ${pi/2}" xyz="0 0 -0.003"/>
-      <geometry>
-        <mesh filename="package://hawaii_descriptions/meshes/vx300_2_shoulder.stl" scale="0.001 0.001 0.001"/>
+      <origin
+        rpy="0 0 ${pi/2}"
+        xyz="0 0 -0.003"/>
+      <geometry>
+        <mesh
+          filename="${mesh_directory}/shoulder.stl"
+          scale="0.001 0.001 0.001"/>
       </geometry>
       <material name="interbotix_black"/>
     </visual>
     <collision>
-      <origin rpy="0 0 ${pi/2}" xyz="0 0 -0.003"/>
-      <geometry>
-        <mesh filename="package://hawaii_descriptions/meshes/vx300_2_shoulder.stl" scale="0.001 0.001 0.001"/>
+      <origin
+        rpy="0 0 ${pi/2}"
+        xyz="0 0 -0.003"/>
+      <geometry>
+        <mesh
+          filename="${mesh_directory}/shoulder.stl"
+          scale="0.001 0.001 0.001"/>
       </geometry>
     </collision>
     <inertial>
-      <origin rpy="0 0 ${pi/2}" xyz="0.0002592330 -0.0000033552 0.0116129000"/>
-      <mass value="0.798614" />
-      <inertia ixx="0.0009388000" iyy="0.0011380000" izz="0.0012010000" ixy="-0.0000000010" ixz="-0.0000000191" iyz="0.0000059568" />
+      <origin
+        rpy="0 0 ${pi/2}"
+        xyz="0.0002592330 -0.0000033552 0.0116129000"/>
+      <mass value="0.798614"/>
+      <inertia
+        ixx="0.0009388000"
+        iyy="0.0011380000"
+        izz="0.0012010000"
+        ixy="-0.0000000010"
+        ixz="-0.0000000191"
+        iyz="0.0000059568"/>
     </inertial>
   </link>
   <joint name="shoulder" type="revolute">
     <axis xyz="0 1 0"/>
-    <limit effort="20" lower="${radians(-106)}" upper="${radians(72)}" velocity="${pi}"/>
-    <origin rpy="0 0 0" xyz="0 0 0.04805"/>
-    <parent link="$(arg robot_name)/shoulder_link"/>
-    <child link="$(arg robot_name)/upper_arm_link"/>
-    <dynamics friction="0.1"/>
+    <limit
+      effort="${shoulder_limit_effort}"
+      lower="${shoulder_limit_lower}"
+      upper="${shoulder_limit_upper}"
+      velocity="${shoulder_limit_vel}"/>
+    <origin
+      rpy="0 0 0"
+      xyz="0 0 0.04805"/>
+    <parent
+      link="$(arg robot_name)/shoulder_link"/>
+    <child
+      link="$(arg robot_name)/upper_arm_link"/>
+    <dynamics
+      friction="0.1"
+      damping="0.1"/>
   </joint>
-  <transmission name="trans_shoulder">
-    <type>transmission_interface/SimpleTransmission</type>
-    <joint name="shoulder">
-      <hardwareInterface>hardware_interface/EffortJointInterface</hardwareInterface>
-    </joint>
-    <actuator name="shoulder_motor">
-      <mechanicalReduction>1</mechanicalReduction>
-    </actuator>
-  </transmission>
   <link name="$(arg robot_name)/upper_arm_link">
     <visual>
-      <origin rpy="0 0 ${pi/2}" xyz="0 0 0"/>
-      <geometry>
-        <mesh filename="package://hawaii_descriptions/meshes/vx300_3_upper_arm.stl" scale="0.001 0.001 0.001"/>
+      <origin
+        rpy="0 0 ${pi/2}"
+        xyz="0 0 0"/>
+      <geometry>
+        <mesh
+          filename="${mesh_directory}/upper_arm.stl"
+          scale="0.001 0.001 0.001"/>
       </geometry>
       <material name="interbotix_black"/>
     </visual>
     <collision>
-      <origin rpy="0 0 ${pi/2}" xyz="0 0 0"/>
-      <geometry>
-        <mesh filename="package://hawaii_descriptions/meshes/vx300_3_upper_arm.stl" scale="0.001 0.001 0.001"/>
+      <origin
+        rpy="0 0 ${pi/2}"
+        xyz="0 0 0"/>
+      <geometry>
+        <mesh
+          filename="${mesh_directory}/upper_arm.stl"
+          scale="0.001 0.001 0.001"/>
       </geometry>
     </collision>
     <inertial>
-      <origin rpy="0 0 ${pi/2}" xyz="0.0206949000 0.0000000004 0.2264590000"/>
-      <mass value="0.792592" />
-      <inertia ixx="0.0089250000" iyy="0.0089370000" izz="0.0009357000" ixy="0.0000000000" ixz="0.0000000000" iyz="0.0012010000" />
+      <origin
+        rpy="0 0 ${pi/2}"
+        xyz="0.0206949000 0.0000000004 0.2264590000"/>
+      <mass value="0.792592"/>
+      <inertia
+        ixx="0.0089250000"
+        iyy="0.0089370000"
+        izz="0.0009357000"
+        ixy="0.0000000000"
+        ixz="0.0000000000"
+        iyz="0.0012010000"/>
     </inertial>
   </link>
   <joint name="elbow" type="revolute">
     <axis xyz="0 1 0"/>
-    <limit effort="15" lower="${radians(-101)}" upper="${radians(92)}" velocity="${pi}"/>
-    <origin rpy="0 0 0" xyz="0.05955 0 0.3"/>
-    <parent link="$(arg robot_name)/upper_arm_link"/>
-    <child link="$(arg robot_name)/forearm_link"/>
-    <dynamics friction="0.1"/>
+    <limit
+      effort="${elbow_limit_effort}"
+      lower="${elbow_limit_lower}"
+      upper="${elbow_limit_upper}"
+      velocity="${elbow_limit_vel}"/>
+    <origin
+      rpy="0 0 0"
+      xyz="0.05955 0 0.3"/>
+    <parent
+      link="$(arg robot_name)/upper_arm_link"/>
+    <child
+      link="$(arg robot_name)/forearm_link"/>
+    <dynamics
+      friction="0.1"
+      damping="0.1"/>
   </joint>
-  <transmission name="trans_elbow">
-    <type>transmission_interface/SimpleTransmission</type>
-    <joint name="elbow">
-      <hardwareInterface>hardware_interface/EffortJointInterface</hardwareInterface>
-    </joint>
-    <actuator name="elbow_motor">
-      <mechanicalReduction>1</mechanicalReduction>
-    </actuator>
-  </transmission>
   <link name="$(arg robot_name)/forearm_link">
     <visual>
-      <origin rpy="0 0 ${pi/2}" xyz="0 0 0"/>
-      <geometry>
-        <mesh filename="package://hawaii_descriptions/meshes/vx300_4_forearm.stl" scale="0.001 0.001 0.001"/>
+      <origin
+        rpy="0 0 ${pi/2}"
+        xyz="0 0 0"/>
+      <geometry>
+        <mesh
+          filename="${mesh_directory}/forearm.stl"
+          scale="0.001 0.001 0.001"/>
       </geometry>
       <material name="interbotix_black"/>
     </visual>
     <collision>
-      <origin rpy="0 0 ${pi/2}" xyz="0 0 0"/>
-      <geometry>
-        <mesh filename="package://hawaii_descriptions/meshes/vx300_4_forearm.stl" scale="0.001 0.001 0.001"/>
+      <origin
+        rpy="0 0 ${pi/2}"
+        xyz="0 0 0"/>
+      <geometry>
+        <mesh
+          filename="${mesh_directory}/forearm.stl"
+          scale="0.001 0.001 0.001"/>
       </geometry>
     </collision>
     <inertial>
-      <origin rpy="0 0 ${pi/2}" xyz="0.1812650000 -0.0002065037 0.0000000000"/>
-      <mass value="0.544659" />
-      <inertia ixx="0.0054470000" iyy="0.0002267000" izz="0.0055740000" ixy="-0.0000119800" ixz="0.0000000000" iyz="0.0000000000" />
+      <origin
+        rpy="0 0 ${pi/2}"
+        xyz="0.1812650000 -0.0002065037 0.0000000000"/>
+      <mass value="0.544659"/>
+      <inertia
+        ixx="0.0054470000"
+        iyy="0.0002267000"
+        izz="0.0055740000"
+        ixy="-0.0000119800"
+        ixz="0.0000000000"
+        iyz="0.0000000000"/>
     </inertial>
   </link>
   <joint name="wrist_angle" type="revolute">
     <axis xyz="0 1 0"/>
-    <limit effort="5" lower="${radians(-107)}" upper="${radians(128)}" velocity="${pi}"/>
-    <origin rpy="0 0 0" xyz="0.3 0 0"/>
-    <parent link="$(arg robot_name)/forearm_link"/>
-    <child link="$(arg robot_name)/wrist_link"/>
-    <dynamics friction="0.1"/>
+    <limit
+      effort="${wrist_angle_limit_effort}"
+      lower="${wrist_angle_limit_lower}"
+      upper="${wrist_angle_limit_upper}"
+      velocity="${wrist_angle_limit_vel}"/>
+    <origin
+      rpy="0 0 0"
+      xyz="0.3 0 0"/>
+    <parent
+      link="$(arg robot_name)/forearm_link"/>
+    <child
+      link="$(arg robot_name)/wrist_link"/>
+    <dynamics
+      friction="0.1"
+      damping="0.1"/>
   </joint>
-  <transmission name="trans_wrist_angle">
-    <type>transmission_interface/SimpleTransmission</type>
-    <joint name="wrist_angle">
-      <hardwareInterface>hardware_interface/EffortJointInterface</hardwareInterface>
-    </joint>
-    <actuator name="wrist_angle_motor">
-      <mechanicalReduction>1</mechanicalReduction>
-    </actuator>
-  </transmission>
   <link name="$(arg robot_name)/wrist_link">
     <visual>
-      <origin rpy="0 0 ${pi/2}" xyz="0 0 0"/>
-      <geometry>
-        <mesh filename="package://hawaii_descriptions/meshes/vx300_5_wrist.stl" scale="0.001 0.001 0.001"/>
+      <origin
+        rpy="0 0 ${pi/2}"
+        xyz="0 0 0"/>
+      <geometry>
+        <mesh
+          filename="${mesh_directory}/wrist.stl"
+          scale="0.001 0.001 0.001"/>
       </geometry>
       <material name="interbotix_black"/>
     </visual>
     <collision>
-      <origin rpy="0 0 ${pi/2}" xyz="0 0 0"/>
-      <geometry>
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
Commit message: cleaned up hawaii_descriptions and hawaii_gazebo

File: hawaii_ros_ws/src/hawaii_descriptions/urdf/hawaii.urdf.xacro (robot description, xacro)
@@ -13,8 +13,8 @@
   <xacro:arg name="show_gripper_bar"                default="true"/>
   <xacro:arg name="show_gripper_fingers"            default="true"/>
-  <xacro:arg name="use_world_frame"                 default="false"/>
+  <xacro:arg name="use_world_frame"                 default="true"/>
   <xacro:arg name="external_urdf_loc"               default=""/>
   <xacro:arg name="hardware_type"                   default="actual"/>
-  <xacro:property name="mesh_directory"             value="package://hawaii_descriptions/meshes"/>
+  <xacro:property name="mesh_directory"             value="package://hawaii_descriptions/meshes/${robot_model}_meshes/"/>
   <xacro:property name="urdf_loc"                   value="$(arg external_urdf_loc)"/>
   <xacro:property name="hardware_type"              value="$(arg hardware_type)"/>
