Commit message: changed urdf and config file to control dynamixel

File: hawaii_ros_ws/src/hawaii_descriptions/urdf/control.urdf.xacro (robot description, xacro)
@@ -4,12 +4,11 @@
     <hardware>
       <!-- If we are using the actual, physical robot -->
-      <!--<xacro:if value="${hardware_type == 'actual'}">
+      <xacro:if value="${hardware_type == 'actual'}">
         <plugin>interbotix_xs_ros_control/XSHardwareInterface</plugin>
         <param name="loop_hz">10</param>
         <param name="group_name">arm</param>
-        <param name="gripper_name">gripper</param>
+       <!--<param name="gripper_name">gripper</param>-->
         <param name="joint_states_topic">joint_states</param>
       </xacro:if>
-      -->
       <!-- If doing basic simulation of the robot -->
       <xacro:if value="${hardware_type == 'fake'}">
@@ -28,85 +27,4 @@
       <state_interface name="position"/>
     </joint>
-    <joint name="shoulder">
-      <command_interface name="position">
-        <param name="min">"${shoulder_limit_lower}"</param>
-        <param name="max">"${shoulder_limit_upper}"</param>
-      </command_interface>
-      <state_interface name="position"/>
-    </joint>
-    <joint name="elbow">
-      <command_interface name="position">
-        <param name="min">"${elbow_limit_lower}"</param>
-        <param name="max">"${elbow_limit_upper}"</param>
-      </command_interface>
-      <state_interface name="position"/>
-    </joint>
-    <xacro:if value="${dof >= 6}">
-      <joint name="forearm_roll">
-        <command_interface name="position">
-          <param name="min">"${forearm_roll_limit_lower}"</param>
-          <param name="max">"${forearm_roll_limit_upper}"</param>
-        </command_interface>
-        <state_interface name="position"/>
-      </joint>
-    </xacro:if>
-    <joint name="wrist_angle">
-      <command_interface name="position">
-        <param name="min">"${wrist_angle_limit_lower}"</param>
-        <param name="max">"${wrist_angle_limit_upper}"</param>
-      </command_interface>
-      <state_interface name="position"/>
-    </joint>
-    <xacro:if value="${dof >= 5}">
-      <joint name="wrist_rotate">
-        <command_interface name="position">
-          <param name="min">"${wrist_rotate_limit_lower}"</param>
-          <param name="max">"${wrist_rotate_limit_upper}"</param>
-        </command_interface>
-        <state_interface name="position"/>
-      </joint>
-    </xacro:if>
-    <xacro:if value="$(arg use_gripper)">
-      <xacro:if value="${hardware_type in ('fake', 'gz_classic')}">
-        <joint name="gripper">
-          <command_interface name="position"/>
-          <state_interface name="position"/>
-        </joint>
-      </xacro:if>
-      <xacro:if value="$(arg show_gripper_fingers)">
-        <joint name="left_finger">
-          <command_interface name="position">
-            <param name="min">"${finger_limit_lower}"</param>
-            <param name="max">"${-finger_limit_lower}"</param>
-          </command_interface>
-          <state_interface name="position"/>
-        </joint>
-        <xacro:if value="${hardware_type == 'gz_classic'}">
-          <joint name="right_finger">
-            <!-- <param name="mimic">left_finger</param>
-            <param name="multiplier">1</param> -->
-            <command_interface name="position">
-              <param name="min">"${-finger_limit_lower}"</param>
-              <param name="max">"${finger_limit_lower}"</param>
-            </command_interface>
-            <state_interface name="position"/>
-          </joint>
-        </xacro:if>
-      </xacro:if>
-    </xacro:if>
   </ros2_control>
-  <!-- Load the gazebo_ros2_control plugin if using Gazebo hardware -->
-  <xacro:if value="${hardware_type == 'gz_classic'}">
-    <gazebo>
-      <plugin filename="libgazebo_ros2_control.so" name="gazebo_ros2_control">
-        <ros>
-          <namespace>/$(arg robot_name)</namespace>
-        </ros>
-        <robot_param>robot_description</robot_param>
-        <robot_param_node>robot_state_publisher</robot_param_node>
-        <parameters>$(find hawaii_gazebo)/config/trajectory_controllers/hawaii_trajectory_controllers.yaml</parameters>
-      </plugin>
-    </gazebo>
-    <xacro:include filename="$(find hawaii_gazebo)/media/materials/scripts/interbotix_black.material"/>
-  </xacro:if>
 </robot>

File: hawaii_ros_ws/src/hawaii_descriptions/urdf/hawaii.urdf.xacro (robot description, xacro)
@@ -147,516 +147,5 @@
     </inertial>
   </link>
-  <joint name="shoulder" type="revolute">
-    <axis xyz="0 1 0"/>
-    <limit
-      effort="${shoulder_limit_effort}"
-      lower="${shoulder_limit_lower}"
-      upper="${shoulder_limit_upper}"
-      velocity="${shoulder_limit_vel}"/>
-    <origin
-      rpy="0 0 0"
-      xyz="0 0 0.04805"/>
-    <parent
-      link="$(arg robot_name)/shoulder_link"/>
-    <child
-      link="$(arg robot_name)/upper_arm_link"/>
-    <dynamics
-      friction="0.1"
-      damping="0.1"/>
-  </joint>
-  <link name="$(arg robot_name)/upper_arm_link">
-    <visual>
-      <origin
-        rpy="0 0 ${pi/2}"
-        xyz="0 0 0"/>
-      <geometry>
-        <mesh
-          filename="${mesh_directory}/upper_arm.stl"
-          scale="0.001 0.001 0.001"/>
-      </geometry>
-      <material name="interbotix_black"/>
-    </visual>
-    <collision>
-      <origin
-        rpy="0 0 ${pi/2}"
-        xyz="0 0 0"/>
-      <geometry>
-        <mesh
-          filename="${mesh_directory}/upper_arm.stl"
-          scale="0.001 0.001 0.001"/>
-      </geometry>
-    </collision>
-    <inertial>
-      <origin
-        rpy="0 0 ${pi/2}"
-        xyz="0.0206949000 0.0000000004 0.2264590000"/>
-      <mass value="0.792592"/>
-      <inertia
-        ixx="0.0089250000"
-        iyy="0.0089370000"
-        izz="0.0009357000"
-        ixy="0.0000000000"
-        ixz="0.0000000000"
-        iyz="0.0012010000"/>
-    </inertial>
-  </link>
-  <joint name="elbow" type="revolute">
-    <axis xyz="0 1 0"/>
-    <limit
-      effort="${elbow_limit_effort}"
-      lower="${elbow_limit_lower}"
-      upper="${elbow_limit_upper}"
-      velocity="${elbow_limit_vel}"/>
-    <origin
-      rpy="0 0 0"
-      xyz="0.05955 0 0.3"/>
-    <parent
-      link="$(arg robot_name)/upper_arm_link"/>
-    <child
-      link="$(arg robot_name)/forearm_link"/>
-    <dynamics
-      friction="0.1"
-      damping="0.1"/>
-  </joint>
-  <link name="$(arg robot_name)/forearm_link">
-    <visual>
-      <origin
-        rpy="0 0 ${pi/2}"
-        xyz="0 0 0"/>
-      <geometry>
-        <mesh
-          filename="${mesh_directory}/forearm.stl"
-          scale="0.001 0.001 0.001"/>
-      </geometry>
-      <material name="interbotix_black"/>
-    </visual>
-    <collision>
-      <origin
-        rpy="0 0 ${pi/2}"
-        xyz="0 0 0"/>
-      <geometry>
-        <mesh
-          filename="${mesh_directory}/forearm.stl"
-          scale="0.001 0.001 0.001"/>
-      </geometry>
-    </collision>
-    <inertial>
-      <origin
-        rpy="0 0 ${pi/2}"
-        xyz="0.1812650000 -0.0002065037 0.0000000000"/>
-      <mass value="0.544659"/>
-      <inertia
-        ixx="0.0054470000"
-        iyy="0.0002267000"
-        izz="0.0055740000"
-        ixy="-0.0000119800"
-        ixz="0.0000000000"
-        iyz="0.0000000000"/>
-    </inertial>
-  </link>
-  <joint name="wrist_angle" type="revolute">
-    <axis xyz="0 1 0"/>
-    <limit
-      effort="${wrist_angle_limit_effort}"
-      lower="${wrist_angle_limit_lower}"
-      upper="${wrist_angle_limit_upper}"
-      velocity="${wrist_angle_limit_vel}"/>
-    <origin
-      rpy="0 0 0"
-      xyz="0.3 0 0"/>
-    <parent
-      link="$(arg robot_name)/forearm_link"/>
-    <child
-      link="$(arg robot_name)/wrist_link"/>
-    <dynamics
-      friction="0.1"
-      damping="0.1"/>
-  </joint>
-  <link name="$(arg robot_name)/wrist_link">
-    <visual>
-      <origin
-        rpy="0 0 ${pi/2}"
-        xyz="0 0 0"/>
-      <geometry>
-        <mesh
-          filename="${mesh_directory}/wrist.stl"
-          scale="0.001 0.001 0.001"/>
-      </geometry>
-      <material name="interbotix_black"/>
-    </visual>
-    <collision>
-      <origin
-        rpy="0 0 ${pi/2}"
-        xyz="0 0 0"/>
-      <geometry>
-        <mesh
-          filename="${mesh_directory}/wrist.stl"
-          scale="0.001 0.001 0.001"/>
-      </geometry>
-    </collision>
-    <inertial>
-      <origin
-        rpy="0 0 ${pi/2}"
-        xyz="0.0467430000 -0.0000076652 0.0105650000"/>
-      <mass value="0.115395"/>
-      <inertia
-        ixx="0.0000463100"
-        iyy="0.0000451400"
-        izz="0.0000527000"
-        ixy="0.0000000195"
-        ixz="0.0000000023"
-        iyz="0.0000042002"/>
-    </inertial>
-  </link>
-  <!-- Include the gripper if used -->
-  <xacro:if value="$(arg use_gripper)">
-    <joint name="wrist_rotate" type="revolute">
-      <axis xyz="1 0 0"/>
-      <limit
-        effort="${wrist_rotate_limit_effort}"
-        lower="${wrist_rotate_limit_lower}"
-        upper="${wrist_rotate_limit_upper}"
-        velocity="${wrist_rotate_limit_vel}"/>
-      <origin
-        rpy="0 0 0"
-        xyz="0.069744 0 0"/>
-      <parent
-        link="$(arg robot_name)/wrist_link"/>
-      <child
-        link="$(arg robot_name)/gripper_link"/>
-      <dynamics
-        friction="0.1"
-        damping="0.1"/>
-    </joint>
-    <link name="$(arg robot_name)/gripper_link">
-      <visual>
-        <origin
-          rpy="0 0 ${pi/2}"
-          xyz="-0.02 0 0"/>
-        <geometry>
-          <mesh
-            filename="${mesh_directory}/gripper.stl"
-            scale="0.001 0.001 0.001"/>
-        </geometry>
-        <material name="interbotix_black"/>
-      </visual>
-      <collision>
-        <origin
-          rpy="0 0 ${pi/2}"
-          xyz="-0.02 0 0"/>
-        <geometry>
-          <mesh
-            filename="${mesh_directory}/gripper.stl"
-            scale="0.001 0.001 0.001"/>
-        </geometry>
-      </collision>
-      <inertial>
-        <origin
-          rpy="0 0 ${pi/2}"
-          xyz="0.0230010000 0.0000000000 0.0115230000"/>
-        <mass value="0.097666"/>
-        <inertia
-          ixx="0.0000326800"
-          iyy="0.0000243600"
-          izz="0.0000211900"
-          ixy="0.0000000000"
-          ixz="0.0000000000"
-          iyz="0.0000002785"/>
-      </inertial>
-    </link>
-    <joint name="ee_arm" type="fixed">
-      <axis xyz="1 0 0"/>
-      <origin
-        rpy="0 0 0"
-        xyz="0.042825 0 0"/>
-      <parent
-        link="$(arg robot_name)/gripper_link"/>
-      <child
-        link="$(arg robot_name)/ee_arm_link"/>
-    </joint>
-    <link name="$(arg robot_name)/ee_arm_link">
-      <inertial>
-        <mass value="0.001"/>
-        <inertia
-          ixx="0.0001"
-          iyy="0.0001"
-          izz="0.0001"
-          ixy="0"
-          ixz="0"
-          iyz="0"/>
-      </inertial>
-    </link>
-    <joint name="gripper" type="continuous">
-      <axis xyz="1 0 0"/>
-      <limit
-        effort="1"
-        velocity="${gripper_limit_vel}"/>
-      <origin
-        rpy="0 0 0"
-        xyz="0.005675 0 0"/>
-      <parent
-        link="$(arg robot_name)/ee_arm_link"/>
-      <child
-        link="$(arg robot_name)/gripper_prop_link"/>
-      <dynamics
-        friction="0.1"
-        damping="0.1"/>
-    </joint>
-    <link name="$(arg robot_name)/gripper_prop_link">
-      <visual>
-        <origin
-          rpy="0 0 ${pi/2}"
-          xyz="-0.0685 0 0"/>
-        <geometry>
-          <mesh
-            filename="${mesh_directory}/gripper_prop.stl"
-            scale="0.001 0.001 0.001"/>
-        </geometry>
-        <material name="interbotix_black"/>
-      </visual>
-      <collision>
-        <origin
-          rpy="0 0 ${pi/2}"
-          xyz="-0.0685 0 0"/>
-        <geometry>
-          <mesh
-            filename="${mesh_directory}/gripper_prop.stl"
-            scale="0.001 0.001 0.001"/>
-        </geometry>
-      </collision>
-      <inertial>
-        <origin
-          rpy="0 0 ${pi/2}"
-          xyz="0.0023780000 0.0000000285 0.0000000000"/>
-        <mass value="0.008009"/>
-        <inertia
-          ixx="0.0000020386"
-          iyy="0.0000042979"
-          izz="0.0000023796"
-          ixy="0.0000000000"
-          ixz="0.0000006559"
-          iyz="0.0000000000"/>
-      </inertial>
-    </link>
-    <!-- If the AR tag is being used, then add the AR tag mount -->
-    <xacro:if value="$(arg show_ar_tag)">
-      <xacro:include filename="$(find hawaii_descriptions)/urdf/ar_tag.urdf.xacro"/>
-    </xacro:if> <!-- show_ar_tag -->
-    <!-- If the gripper bar is being used, then also add the gripper bar -->
-    <xacro:if value="$(arg show_gripper_bar)">
-      <joint name="gripper_bar" type="fixed">
-        <axis xyz="1 0 0"/>
-        <origin
-          rpy="0 0 0"
-          xyz="0 0 0"/>
-        <parent
-          link="$(arg robot_name)/ee_arm_link"/>
-        <child
-          link="$(arg robot_name)/gripper_bar_link"/>
-      </joint>
-      <link name="$(arg robot_name)/gripper_bar_link">
-        <visual>
-          <origin
-            rpy="0 0 ${pi/2}"
-            xyz="-0.063 0 0"/>
-          <geometry>
-            <mesh
-              filename="${mesh_directory}/gripper_bar.stl"
-              scale="0.001 0.001 0.001"/>
-          </geometry>
-          <material name="interbotix_black"/>
-        </visual>
-        <collision>
-          <origin
-            rpy="0 0 ${pi/2}"
-            xyz="-0.063 0 0"/>
-          <geometry>
-            <mesh
-              filename="${mesh_directory}/gripper_bar.stl"
-              scale="0.001 0.001 0.001"/>
-          </geometry>
-        </collision>
-        <inertial>
-          <origin
-            rpy="0 0 ${pi/2}"
-            xyz="0.0067940000 -0.0000004272 -0.0007760000"/>
-          <mass value="0.150986"/>
-          <inertia
-            ixx="0.0000789500"
-            iyy="0.0003283000"
-            izz="0.0003095000"
-            ixy="-0.0000000012"
-            ixz="0.0000001341"
-            iyz="0.0000017465"/>
-        </inertial>
-      </link>
-      <joint name="ee_bar" type="fixed">
-        <axis xyz="1 0 0"/>
-        <origin
-          rpy="0 0 0"
-          xyz="0.025875 0 0"/>
-        <parent
-          link="$(arg robot_name)/gripper_bar_link"/>
-        <child
-          link="$(arg robot_name)/fingers_link"/>
-      </joint>
-      <link name="$(arg robot_name)/fingers_link">
-        <inertial>
-          <mass value="0.001"/>
-          <inertia
-            ixx="0.0001"
-            iyy="0.0001"
-            izz="0.0001"
-            ixy="0"
-            ixz="0"
-            iyz="0"/>
-        </inertial>
-      </link>
-      <!-- If the gripper fingers are being used, add those as well -->
-      <xacro:if value="$(arg show_gripper_fingers)">
-        <joint name="left_finger" type="prismatic">
-          <axis xyz="0 1 0"/>
-          <limit
-            effort="${finger_limit_effort}"
-            lower="${finger_limit_lower}"
-            upper="${finger_limit_upper}"
-            velocity="${finger_limit_vel}"/>
-          <origin
-            rpy="0 0 0"
-            xyz="0 0 0"/>
-          <parent
-            link="$(arg robot_name)/fingers_link"/>
-          <child
-            link="$(arg robot_name)/left_finger_link"/>
-          <dynamics
-            friction="0.1"
-            damping="0.1"/>
-        </joint>
-        <link name="$(arg robot_name)/left_finger_link">
-          <visual>
-            <origin
-              rpy="${pi/2} ${-pi} ${pi/2}"
-              xyz="-0.0404 -0.0575 0"/>
-            <geometry>
-              <mesh
-                filename="${mesh_directory}/gripper_finger.stl"
-                scale="0.001 0.001 0.001"/>
-            </geometry>
-            <material name="interbotix_black"/>
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