Commit message: update mode and motor configs for student arm urdf, also created script to generate kinematics matrices from urdf file

File: hawaii_ros_ws/src/hawaii_descriptions/urdf/Student_Arm.urdf (robot description, URDF)
Before this commit: robot hawaii, 10 links, 9 joints
Links:
- link Gripper_Left: geometry collision mesh filename=../meshes/hawaii_meshes/Gripper_Left.STL; visual mesh filename=../meshes/hawaii_meshes/Gripper_Left.STL
- link Gripper_Right: geometry collision mesh filename=../meshes/hawaii_meshes/Gripper_Right.STL; visual mesh filename=../meshes/hawaii_meshes/Gripper_Right.STL
- link J1: geometry collision mesh filename=../meshes/hawaii_meshes/J1.STL; visual mesh filename=../meshes/hawaii_meshes/J1.STL
- link J2: geometry collision mesh filename=../meshes/hawaii_meshes/J2.STL; visual mesh filename=../meshes/hawaii_meshes/J2.STL
- link J3: geometry collision mesh filename=../meshes/hawaii_meshes/J3.STL; visual mesh filename=../meshes/hawaii_meshes/J3.STL
- link J4: geometry collision mesh filename=../meshes/hawaii_meshes/J4.STL; visual mesh filename=../meshes/hawaii_meshes/J4.STL
- link J5: geometry collision mesh filename=../meshes/hawaii_meshes/J5.STL; visual mesh filename=../meshes/hawaii_meshes/J5.STL
- link J6: geometry collision mesh filename=../meshes/hawaii_meshes/J6.STL; visual mesh filename=../meshes/hawaii_meshes/J6.STL
- link base_link: geometry collision mesh filename=../meshes/hawaii_meshes/base_link.STL; visual mesh filename=../meshes/hawaii_meshes/base_link.STL
Joints:
- joint GL: limit lower=${GL_limit_lower} upper=${GL_limit_upper} effort=${GL_limit_effort} velocity=${GL_limit_vel} -> lower=0 upper=0.057 effort=0 velocity=0
- joint GR: limit lower=${GR_limit_lower} upper=${GR_limit_upper} effort=${GR_limit_effort} velocity=${GR_limit_vel} -> lower=0 upper=0.057 effort=0 velocity=0
- joint J1: limit lower=${J1_limit_lower} upper=${J1_limit_upper} effort=${J1_limit_effort} velocity=${J1_limit_vel} -> lower=0 upper=0 effort=0 velocity=0
- joint J2: limit lower=${J2_limit_lower} upper=${J2_limit_upper} effort=${J2_limit_effort} velocity=${J2_limit_vel} -> lower=-1.4 upper=2.5 effort=0 velocity=0
- joint J3: limit lower=${J3_limit_lower} upper=${J3_limit_upper} effort=${J3_limit_effort} velocity=${J3_limit_vel} -> lower=-1.4 upper=1.8 effort=0 velocity=0
- joint J5: limit lower=${J5_limit_lower} upper=${J5_limit_upper} effort=${J5_limit_effort} velocity=${J5_limit_vel} -> lower=-0.75 upper=2.9 effort=0 velocity=0

Commit message: Working control of joints through ARM API, grippers still need work. updated limits and joint types in urdf, updated kinematics in mr_descriptions

File: hawaii_ros_ws/src/hawaii_descriptions/urdf/Student_Arm.urdf (robot description, URDF)
Before this commit: robot Student_Arm, 10 links, 9 joints
Joints:
- joint J1: limit lower=0 upper=0 effort=0 velocity=0 -> lower=-3.141592653589793 upper=3.141592653589793 effort=0 velocity=0; type continuous -> revolute
- joint J4: limit (none) -> lower=-3.141592653589793 upper=3.141592653589793 effort=0 velocity=0; type continuous -> revolute
- joint J6: limit (none) -> lower=-3.141592653589793 upper=3.141592653589793 effort=0 velocity=0; type continuous -> revolute

File: hawaii_ros_ws/src/hawaii_descriptions/urdf/Student_Arm.urdf.xacro (robot description, xacro)
@@ -1,21 +1,21 @@
 <?xml version="1.0"?>
-<robot name="hawaii" xmlns:xacro="http://ros.org/wiki/xacro">
+<robot name="Student_Arm" xmlns:xacro="http://ros.org/wiki/xacro">
   <xacro:property name="pi_offset"                  value="0.00001"/>
   <xacro:property name="J1_limit_effort"            value="0"/>
-  <xacro:property name="J1_limit_lower"             value="0"/>
-  <xacro:property name="J1_limit_upper"             value="0"/>
-  <xacro:property name="J1_limit_vel"               value="0"/>
+  <xacro:property name="J1_limit_lower"             value="-3.141592653589793"/>
+  <xacro:property name="J1_limit_upper"             value="3.141592653589793"/>
+  <xacro:property name="J1_limit_vel"               value="3.141592653589793"/>
   <xacro:property name="J2_limit_effort"            value="0"/>
   <xacro:property name="J2_limit_lower"             value="${radians(-80)}"/>
   <xacro:property name="J2_limit_upper"             value="${radians(143)}"/>
-  <xacro:property name="J2_limit_vel"               value="0"/>
+  <xacro:property name="J2_limit_vel"               value="3.141592653589793"/>
   <xacro:property name="J3_limit_effort"            value="0"/>
   <xacro:property name="J3_limit_lower"             value="-1.4"/>
   <xacro:property name="J3_limit_upper"             value="1.8"/>
-  <xacro:property name="J3_limit_vel"               value="0"/>
+  <xacro:property name="J3_limit_vel"               value="3.141592653589793"/>
   <xacro:property name="J5_limit_effort"            value="0"/>
   <xacro:property name="J5_limit_lower"             value="-0.75"/>
   <xacro:property name="J5_limit_upper"             value="2.9"/>
-  <xacro:property name="J5_limit_vel"               value="0"/>
+  <xacro:property name="J5_limit_vel"               value="3.141592653589793"/>
   <xacro:property name="GR_limit_effort"            value="0"/>
   <xacro:property name="GR_limit_lower"             value="0"/>
@@ -110,5 +110,5 @@
   </link>
   <joint name="J1"
-    type="continuous">
+    type="revolute">
     <origin
       xyz="0 0 0"
@@ -283,5 +283,5 @@
   <joint
     name="J4"
-    type="continuous">
+    type="revolute">
     <origin
       xyz="0 -0.232125103077643 0.0220999999999999"
@@ -293,4 +293,9 @@
     <axis
       xyz="0 0.707106781186543 -0.707106781186552" />
+    <limit
+      effort="0"
+      lower="-3.141592653589793"
+      upper="3.141592653589793"
+      velocity="3.141592653589793"/>
   </joint>
   <link
@@ -394,5 +399,5 @@
   <joint
     name="J6"
-    type="continuous">
+    type="revolute">
     <origin
       xyz="-0.0410888768161758 0.0397298912546164 0"
@@ -404,4 +409,9 @@
     <axis
       xyz="0 0 1" />
+    <limit
+      effort="0"
+      lower="-3.141592653589793"
+      upper="3.141592653589793"
+      velocity="3.141592653589793"/>
   </joint>
   <link

Commit message: added gripper joint to urdf, and config files, and updated sdk sim script to work with this type of gripper

File: hawaii_ros_ws/src/hawaii_descriptions/urdf/Student_Arm.urdf (robot description, URDF)
Before this commit: robot Student_Arm, 10 links, 9 joints
Links:
- added link finger_link, mass 0.001
Joints:
- added joint gripper: type fixed, parent J6, child finger_link, origin xyz=0 0 0 rpy=0 0 0, axis 1 0 0
- joint GL: parent J6 -> finger_link
- joint GR: limit lower=0 upper=0.057 effort=0 velocity=0 -> lower=-0.057 upper=0 effort=0 velocity=0; parent J6 -> finger_link

File: hawaii_ros_ws/src/hawaii_descriptions/urdf/Student_Arm.urdf.xacro (robot description, xacro)
@@ -18,12 +18,12 @@
   <xacro:property name="J5_limit_upper"             value="2.9"/>
   <xacro:property name="J5_limit_vel"               value="3.141592653589793"/>
-  <xacro:property name="GR_limit_effort"            value="0"/>
-  <xacro:property name="GR_limit_lower"             value="0"/>
-  <xacro:property name="GR_limit_upper"             value="0.057"/>
-  <xacro:property name="GR_limit_vel"               value="0"/>
-  <xacro:property name="GL_limit_effort"            value="0"/>
+  <xacro:property name="GR_limit_effort"            value="5"/>
+  <xacro:property name="GR_limit_lower"             value="-0.057"/>
+  <xacro:property name="GR_limit_upper"             value="0"/>
+  <xacro:property name="GR_limit_vel"               value="1"/>
+  <xacro:property name="GL_limit_effort"            value="5"/>
   <xacro:property name="GL_limit_lower"             value="0"/>
   <xacro:property name="GL_limit_upper"             value="0.057"/>
-  <xacro:property name="GL_limit_vel"               value="0"/>
+  <xacro:property name="GL_limit_vel"               value="1"/>
   <link name="world"/>
   <joint name="fixed" type="fixed">
@@ -462,5 +462,5 @@
       rpy="0 0 1.97991331761951" />
     <parent
-      link="J6" />
+      link="finger_link" />
     <child
       link="Gripper_Left" />
@@ -520,5 +520,5 @@
       rpy="-1.5707963267949 0 -2.73247566276518" />
     <parent
-      link="J6" />
+      link="finger_link" />
     <child
       link="Gripper_Right" />
@@ -535,3 +535,28 @@
       offset="0" />
   </joint>
+  <joint
+    name="gripper"
+    type="fixed">
+    <origin
+      xyz="0 0 0"
+      rpy="0 0 0" />
+    <parent
+      link="J6" />
+    <child
+      link="finger_link" />
+    <axis
+      xyz="1 0 0" />
+  </joint>
+  <link name="finger_link">
+          <inertial>
+            <mass value="0.001"/>
+            <inertia
+              ixx="0.0001"
+              iyy="0.0001"
+              izz="0.0001"
+              ixy="0"
+              ixz="0"
+              iyz="0"/>
+          </inertial>
+        </link>
 </robot>
