Commit message: fixed student arm urdf and put Slist and M matrices into mr_descriptions

File: hawaii_ros_ws/src/hawaii_descriptions/urdf/Student_Arm.urdf.xacro (robot description, xacro)
@@ -23,7 +23,7 @@
   <xacro:property name="GR_limit_vel"               value="0"/>
   <xacro:property name="GL_limit_effort"            value="0"/>
-  <xacro:property name="GR_limit_lower"             value="0"/>
-  <xacro:property name="GR_limit_upper"             value="0.057"/>
-  <xacro:property name="GR_limit_vel"               value="0"/>
+  <xacro:property name="GL_limit_lower"             value="0"/>
+  <xacro:property name="GL_limit_upper"             value="0.057"/>
+  <xacro:property name="GL_limit_vel"               value="0"/>
   <link name="world"/>
   <joint name="fixed" type="fixed">

Commit message: fixing GR limits

File: hawaii_ros_ws/src/hawaii_descriptions/urdf/Student_Arm.urdf.xacro (robot description, xacro)
@@ -19,6 +19,6 @@
   <xacro:property name="J5_limit_vel"               value="3.141592653589793"/>
   <xacro:property name="GR_limit_effort"            value="5"/>
-  <xacro:property name="GR_limit_lower"             value="-0.057"/>
-  <xacro:property name="GR_limit_upper"             value="0"/>
+  <xacro:property name="GR_limit_lower"             value="0"/>
+  <xacro:property name="GR_limit_upper"             value="0.057"/>
   <xacro:property name="GR_limit_vel"               value="1"/>
   <xacro:property name="GL_limit_effort"            value="5"/>

Commit message: cleaning up urdf

File: hawaii_ros_ws/src/hawaii_descriptions/urdf/Student_Arm.urdf.xacro (robot description, xacro)
@@ -1,21 +1,28 @@
 <?xml version="1.0"?>
 <robot name="Student_Arm" xmlns:xacro="http://ros.org/wiki/xacro">
-  <xacro:property name="pi_offset"                  value="0.00001"/>
   <xacro:property name="J1_limit_effort"            value="0"/>
-  <xacro:property name="J1_limit_lower"             value="-3.141592653589793"/>
-  <xacro:property name="J1_limit_upper"             value="3.141592653589793"/>
-  <xacro:property name="J1_limit_vel"               value="3.141592653589793"/>
+  <xacro:property name="J1_limit_lower"             value="${-pi}"/>
+  <xacro:property name="J1_limit_upper"             value="${pi}"/>
+  <xacro:property name="J1_limit_vel"               value="${pi}"/>
   <xacro:property name="J2_limit_effort"            value="0"/>
   <xacro:property name="J2_limit_lower"             value="${radians(-80)}"/>
   <xacro:property name="J2_limit_upper"             value="${radians(143)}"/>
-  <xacro:property name="J2_limit_vel"               value="3.141592653589793"/>
+  <xacro:property name="J2_limit_vel"               value="${pi}"/>
   <xacro:property name="J3_limit_effort"            value="0"/>
   <xacro:property name="J3_limit_lower"             value="-1.4"/>
   <xacro:property name="J3_limit_upper"             value="1.8"/>
-  <xacro:property name="J3_limit_vel"               value="3.141592653589793"/>
+  <xacro:property name="J3_limit_vel"               value="${pi}"/>
+  <xacro:property name="J4_limit_effort"            value="0"/>
+  <xacro:property name="J4_limit_lower"             value="${-pi}"/>
+  <xacro:property name="J4_limit_upper"             value="${pi}"/>
+  <xacro:property name="J4_limit_vel"               value="${pi}"/>
   <xacro:property name="J5_limit_effort"            value="0"/>
   <xacro:property name="J5_limit_lower"             value="-0.75"/>
   <xacro:property name="J5_limit_upper"             value="2.9"/>
-  <xacro:property name="J5_limit_vel"               value="3.141592653589793"/>
+  <xacro:property name="J5_limit_vel"               value="${pi}"/>
+  <xacro:property name="J6_limit_effort"            value="0"/>
+  <xacro:property name="J6_limit_lower"             value="${-pi}"/>
+  <xacro:property name="J6_limit_upper"             value="${pi}"/>
+  <xacro:property name="J6_limit_vel"               value="${pi}"/>
   <xacro:property name="GR_limit_effort"            value="5"/>
   <xacro:property name="GR_limit_lower"             value="0"/>
@@ -294,8 +301,8 @@
       xyz="0 0.707106781186543 -0.707106781186552" />
     <limit
-      effort="0"
-      lower="-3.141592653589793"
-      upper="3.141592653589793"
-      velocity="3.141592653589793"/>
+      effort="${J4_limit_effort}"
+      lower="${J4_limit_lower}"
+      upper="${J4_limit_upper}"
+      velocity="${J4_limit_vel}"/>
   </joint>
   <link
@@ -410,8 +417,8 @@
       xyz="0 0 1" />
     <limit
-      effort="0"
-      lower="-3.141592653589793"
-      upper="3.141592653589793"
-      velocity="3.141592653589793"/>
+      effort="${J6_limit_effort}"
+      lower="${J6_limit_lower}"
+      upper="${J6_limit_upper}"
+      velocity="${J6_limit_vel}"/>
   </joint>
   <link

Commit message: WIP

File: hawaii_ros_ws/src/hawaii_descriptions/urdf/Student_Arm.urdf.xacro (robot description, xacro)
@@ -1,4 +1,5 @@
 <?xml version="1.0"?>
 <robot name="Student_Arm" xmlns:xacro="http://ros.org/wiki/xacro">
+  <xacro:property name="robot_name"                 default="Student_Arm"/>
   <xacro:property name="J1_limit_effort"            value="0"/>
   <xacro:property name="J1_limit_lower"             value="${-pi}"/>
@@ -36,7 +37,7 @@
   <joint name="fixed" type="fixed">
     <parent link="world"/>
-    <child link="base_link"/>
-  </joint>
-  <link name="base_link">
+    <child link="$(arg robot_name)/base_link"/>
+  </joint>
+  <link name="$(arg robot_name)/base_link">
     <inertial>
       <origin
@@ -77,5 +78,5 @@
     </collision>
   </link>
-  <link name="J1">
+  <link name="$(arg robot_name)/J1">
     <inertial>
       <origin
@@ -122,7 +123,7 @@
       rpy="1.5708 0 0" />
     <parent
-      link="base_link" />
-    <child
-      link="J1" />
+      link="$(arg robot_name)/base_link" />
+    <child
+      link="$(arg robot_name)/J1" />
     <axis
       xyz="0 1 0" />
@@ -133,5 +134,5 @@
       velocity="${J1_limit_vel}"/>
   </joint>
-  <link name="J2">
+  <link name="$(arg robot_name)/J2">
     <inertial>
       <origin
@@ -179,7 +180,7 @@
       rpy="1.5708 1.0391 1.5708" />
     <parent
-      link="J1" />
-    <child
-      link="J2" />
+      link="$(arg robot_name)/J1" />
+    <child
+      link="$(arg robot_name)/J2" />
     <axis
       xyz="0 0 -1" />
@@ -191,5 +192,5 @@
   </joint>
   <link
-    name="J3">
+    name="$(arg robot_name)/J3">
     <inertial>
       <origin
@@ -237,7 +238,7 @@
       rpy="-3.1416 0 1.8245" />
     <parent
-      link="J2" />
-    <child
-      link="J3" />
+      link="$(arg robot_name)/J2" />
+    <child
+      link="$(arg robot_name)/J3" />
     <axis
       xyz="0 0 1" />
@@ -249,5 +250,5 @@
   </joint>
   <link
-    name="J4">
+    name="$(arg robot_name)/J4">
     <inertial>
       <origin
@@ -295,7 +296,7 @@
       rpy="0.785398163397452 1.5707963267949 0" />
     <parent
-      link="J3" />
-    <child
-      link="J4" />
+      link="$(arg robot_name)/J3" />
+    <child
+      link="$(arg robot_name)/J4" />
     <axis
       xyz="0 0.707106781186543 -0.707106781186552" />
@@ -307,5 +308,5 @@
   </joint>
   <link
-    name="J5">
+    name="$(arg robot_name)/J5">
     <inertial>
       <origin
@@ -353,7 +354,7 @@
       rpy="1.5708 0.80221 1.5708" />
     <parent
-      link="J4" />
-    <child
-      link="J5" />
+      link="$(arg robot_name)/J4" />
+    <child
+      link="$(arg robot_name)/J5" />
     <axis
       xyz="0 0 1" />
@@ -365,5 +366,5 @@
   </joint>
   <link
-    name="J6">
+    name="$(arg robot_name)/J6">
     <inertial>
       <origin
@@ -411,7 +412,7 @@
       rpy="1.5707963267949 0.409116990824611 -2.33938085233866" />
     <parent
-      link="J5" />
-    <child
-      link="J6" />
+      link="$(arg robot_name)/J5" />
+    <child
+      link="$(arg robot_name)/J6" />
     <axis
       xyz="0 0 1" />
@@ -423,5 +424,5 @@
   </joint>
   <link
-    name="Gripper_Left">
+    name="$(arg robot_name)/Gripper_Left">
     <inertial>
       <origin
@@ -469,7 +470,7 @@
       rpy="0 0 1.97991331761951" />
     <parent
-      link="finger_link" />
-    <child
-      link="Gripper_Left" />
+      link="$(arg robot_name)/finger_link" />
+    <child
+      link="$(arg robot_name)/Gripper_Left" />
     <axis
       xyz="1 0 0" />
@@ -481,5 +482,5 @@
   </joint>
   <link
-    name="Gripper_Right">
+    name="$(arg robot_name)/Gripper_Right">
     <inertial>
       <origin
@@ -527,7 +528,7 @@
       rpy="-1.5707963267949 0 -2.73247566276518" />
     <parent
-      link="finger_link" />
-    <child
-      link="Gripper_Right" />
+      link="$(arg robot_name)/finger_link" />
+    <child
+      link="$(arg robot_name)/Gripper_Right" />
     <axis
       xyz="0 0 1" />
@@ -549,21 +550,21 @@
       rpy="0 0 0" />
     <parent
-      link="J6" />
-    <child
-      link="finger_link" />
+      link="$(arg robot_name)/J6" />
+    <child
+      link="$(arg robot_name)/finger_link" />
     <axis
       xyz="1 0 0" />
   </joint>
-  <link name="finger_link">
-          <inertial>
-            <mass value="0.001"/>
-            <inertia
-              ixx="0.0001"
-              iyy="0.0001"
-              izz="0.0001"
-              ixy="0"
-              ixz="0"
-              iyz="0"/>
-          </inertial>
-        </link>
+  <link name="$(arg robot_name)/finger_link">
+  <inertial>
+    <mass value="0.001"/>
+    <inertia
+      ixx="0.0001"
+      iyy="0.0001"
+      izz="0.0001"
+      ixy="0"
+      ixz="0"
+      iyz="0"/>
+  </inertial>
+  </link>
 </robot>

Commit message: arms showing up in gazebo, had to update gazebo env vars, and change joint names in URDF so they weren't duplicates of link names

File: hawaii_ros_ws/src/hawaii_descriptions/urdf/Student_Arm.urdf.xacro (robot description, xacro)
@@ -37,7 +37,7 @@
   <joint name="fixed" type="fixed">
     <parent link="world"/>
-    <child link="$(arg robot_name)/base_link"/>
-  </joint>
-  <link name="$(arg robot_name)/base_link">
+    <child link="base_link"/>
+  </joint>
+  <link name="base_link">
     <inertial>
       <origin
@@ -78,5 +78,5 @@
     </collision>
   </link>
-  <link name="$(arg robot_name)/J1">
+  <link name="J1">
     <inertial>
       <origin
@@ -117,5 +117,5 @@
     </collision>
   </link>
-  <joint name="J1"
+  <joint name="Joint1"
     type="revolute">
     <origin
@@ -123,7 +123,7 @@
       rpy="1.5708 0 0" />
     <parent
-      link="$(arg robot_name)/base_link" />
-    <child
-      link="$(arg robot_name)/J1" />
+      link="base_link" />
+    <child
+      link="J1" />
     <axis
       xyz="0 1 0" />
@@ -134,5 +134,5 @@
       velocity="${J1_limit_vel}"/>
   </joint>
-  <link name="$(arg robot_name)/J2">
+  <link name="J2">
     <inertial>
       <origin
@@ -174,5 +174,5 @@
   </link>
   <joint
-    name="J2"
+    name="Joint2"
     type="revolute">
     <origin
@@ -180,7 +180,7 @@
       rpy="1.5708 1.0391 1.5708" />
     <parent
-      link="$(arg robot_name)/J1" />
-    <child
-      link="$(arg robot_name)/J2" />
+      link="J1" />
+    <child
+      link="J2" />
     <axis
       xyz="0 0 -1" />
@@ -192,5 +192,5 @@
   </joint>
   <link
-    name="$(arg robot_name)/J3">
+    name="J3">
     <inertial>
       <origin
@@ -232,5 +232,5 @@
   </link>
   <joint
-    name="J3"
+    name="Joint3"
     type="revolute">
     <origin
@@ -238,7 +238,7 @@
       rpy="-3.1416 0 1.8245" />
     <parent
-      link="$(arg robot_name)/J2" />
-    <child
-      link="$(arg robot_name)/J3" />
+      link="J2" />
+    <child
+      link="J3" />
     <axis
       xyz="0 0 1" />
@@ -250,5 +250,5 @@
   </joint>
   <link
-    name="$(arg robot_name)/J4">
+    name="J4">
     <inertial>
       <origin
@@ -290,5 +290,5 @@
   </link>
   <joint
-    name="J4"
+    name="Joint4"
     type="revolute">
     <origin
@@ -296,7 +296,7 @@
       rpy="0.785398163397452 1.5707963267949 0" />
     <parent
-      link="$(arg robot_name)/J3" />
-    <child
-      link="$(arg robot_name)/J4" />
+      link="J3" />
+    <child
+      link="J4" />
     <axis
       xyz="0 0.707106781186543 -0.707106781186552" />
@@ -308,5 +308,5 @@
   </joint>
   <link
-    name="$(arg robot_name)/J5">
+    name="J5">
     <inertial>
       <origin
@@ -348,5 +348,5 @@
   </link>
   <joint
-    name="J5"
+    name="Joint5"
     type="revolute">
     <origin
@@ -354,7 +354,7 @@
       rpy="1.5708 0.80221 1.5708" />
     <parent
-      link="$(arg robot_name)/J4" />
-    <child
-      link="$(arg robot_name)/J5" />
+      link="J4" />
+    <child
+      link="J5" />
     <axis
       xyz="0 0 1" />
@@ -366,5 +366,5 @@
   </joint>
   <link
-    name="$(arg robot_name)/J6">
+    name="J6">
     <inertial>
       <origin
@@ -406,5 +406,5 @@
   </link>
   <joint
-    name="J6"
+    name="Joint6"
     type="revolute">
     <origin
@@ -412,7 +412,7 @@
       rpy="1.5707963267949 0.409116990824611 -2.33938085233866" />
     <parent
-      link="$(arg robot_name)/J5" />
-    <child
-      link="$(arg robot_name)/J6" />
+      link="J5" />
+    <child
+      link="J6" />
     <axis
       xyz="0 0 1" />
@@ -424,5 +424,5 @@
   </joint>
   <link
-    name="$(arg robot_name)/Gripper_Left">
+    name="Gripper_Left">
     <inertial>
       <origin
@@ -470,7 +470,7 @@
       rpy="0 0 1.97991331761951" />
     <parent
-      link="$(arg robot_name)/finger_link" />
-    <child
-      link="$(arg robot_name)/Gripper_Left" />
+      link="finger_link" />
+    <child
+      link="Gripper_Left" />
     <axis
       xyz="1 0 0" />
@@ -482,5 +482,5 @@
   </joint>
   <link
-    name="$(arg robot_name)/Gripper_Right">
+    name="Gripper_Right">
     <inertial>
       <origin
@@ -528,7 +528,7 @@
       rpy="-1.5707963267949 0 -2.73247566276518" />
     <parent
-      link="$(arg robot_name)/finger_link" />
-    <child
-      link="$(arg robot_name)/Gripper_Right" />
+      link="finger_link" />
+    <child
+      link="Gripper_Right" />
     <axis
       xyz="0 0 1" />
@@ -550,11 +550,11 @@
       rpy="0 0 0" />
     <parent
-      link="$(arg robot_name)/J6" />
-    <child
-      link="$(arg robot_name)/finger_link" />
+      link="J6" />
+    <child
+      link="finger_link" />
     <axis
       xyz="1 0 0" />
   </joint>
-  <link name="$(arg robot_name)/finger_link">
+  <link name="finger_link">
   <inertial>
     <mass value="0.001"/>

Commit message: transforms are correct, but arms still flailing in gazebo

File: hawaii_ros_ws/src/hawaii_descriptions/urdf/Student_Arm.urdf.xacro (robot description, xacro)
@@ -37,7 +37,7 @@
   <joint name="fixed" type="fixed">
     <parent link="world"/>
-    <child link="base_link"/>
-  </joint>
-  <link name="base_link">
+    <child link="$(arg robot_name)/base_link"/>
+  </joint>
+  <link name="$(arg robot_name)/base_link">
     <inertial>
       <origin
@@ -78,5 +78,5 @@
     </collision>
   </link>
-  <link name="J1">
+  <link name="$(arg robot_name)/J1">
     <inertial>
       <origin
@@ -123,7 +123,7 @@
       rpy="1.5708 0 0" />
     <parent
-      link="base_link" />
-    <child
-      link="J1" />
+      link="$(arg robot_name)/base_link" />
+    <child
+      link="$(arg robot_name)/J1" />
     <axis
       xyz="0 1 0" />
@@ -134,5 +134,5 @@
       velocity="${J1_limit_vel}"/>
   </joint>
-  <link name="J2">
+  <link name="$(arg robot_name)/J2">
     <inertial>
       <origin
@@ -180,7 +180,7 @@
       rpy="1.5708 1.0391 1.5708" />
     <parent
-      link="J1" />
-    <child
-      link="J2" />
+      link="$(arg robot_name)/J1" />
+    <child
+      link="$(arg robot_name)/J2" />
     <axis
       xyz="0 0 -1" />
@@ -192,5 +192,5 @@
   </joint>
   <link
-    name="J3">
+    name="$(arg robot_name)/J3">
     <inertial>
       <origin
@@ -238,7 +238,7 @@
       rpy="-3.1416 0 1.8245" />
     <parent
-      link="J2" />
-    <child
-      link="J3" />
+      link="$(arg robot_name)/J2" />
+    <child
+      link="$(arg robot_name)/J3" />
     <axis
       xyz="0 0 1" />
@@ -250,5 +250,5 @@
   </joint>
   <link
-    name="J4">
+    name="$(arg robot_name)/J4">
     <inertial>
       <origin
@@ -296,7 +296,7 @@
       rpy="0.785398163397452 1.5707963267949 0" />
     <parent
-      link="J3" />
-    <child
-      link="J4" />
+      link="$(arg robot_name)/J3" />
+    <child
+      link="$(arg robot_name)/J4" />
     <axis
       xyz="0 0.707106781186543 -0.707106781186552" />
@@ -308,5 +308,5 @@
   </joint>
   <link
-    name="J5">
+    name="$(arg robot_name)/J5">
     <inertial>
       <origin
@@ -354,7 +354,7 @@
       rpy="1.5708 0.80221 1.5708" />
     <parent
-      link="J4" />
-    <child
-      link="J5" />
+      link="$(arg robot_name)/J4" />
+    <child
+      link="$(arg robot_name)/J5" />
     <axis
       xyz="0 0 1" />
@@ -366,5 +366,5 @@
   </joint>
   <link
-    name="J6">
+    name="$(arg robot_name)/J6">
     <inertial>
       <origin
@@ -412,7 +412,7 @@
       rpy="1.5707963267949 0.409116990824611 -2.33938085233866" />
     <parent
-      link="J5" />
-    <child
-      link="J6" />
+      link="$(arg robot_name)/J5" />
+    <child
+      link="$(arg robot_name)/J6" />
     <axis
       xyz="0 0 1" />
@@ -424,5 +424,5 @@
   </joint>
   <link
-    name="Gripper_Left">
+    name="$(arg robot_name)/Gripper_Left">
     <inertial>
       <origin
@@ -470,7 +470,7 @@
       rpy="0 0 1.97991331761951" />
     <parent
-      link="finger_link" />
-    <child
-      link="Gripper_Left" />
+      link="$(arg robot_name)/finger_link" />
+    <child
+      link="$(arg robot_name)/Gripper_Left" />
     <axis
       xyz="1 0 0" />
@@ -482,5 +482,5 @@
   </joint>
   <link
-    name="Gripper_Right">
+    name="$(arg robot_name)/Gripper_Right">
     <inertial>
       <origin
@@ -528,7 +528,7 @@
       rpy="-1.5707963267949 0 -2.73247566276518" />
     <parent
-      link="finger_link" />
-    <child
-      link="Gripper_Right" />
+      link="$(arg robot_name)/finger_link" />
+    <child
+      link="$(arg robot_name)/Gripper_Right" />
     <axis
       xyz="0 0 1" />
@@ -550,11 +550,11 @@
       rpy="0 0 0" />
     <parent
-      link="J6" />
-    <child
-      link="finger_link" />
+      link="$(arg robot_name)/J6" />
+    <child
+      link="$(arg robot_name)/finger_link" />
     <axis
       xyz="1 0 0" />
   </joint>
-  <link name="finger_link">
+  <link name="$(arg robot_name)/finger_link">
   <inertial>
     <mass value="0.001"/>

Commit message: updated all joint limits

File: hawaii_ros_ws/src/hawaii_descriptions/urdf/Student_Arm.urdf.xacro (robot description, xacro)
@@ -7,10 +7,10 @@
   <xacro:property name="J1_limit_vel"               value="${pi}"/>
   <xacro:property name="J2_limit_effort"            value="0"/>
-  <xacro:property name="J2_limit_lower"             value="${radians(-80)}"/>
-  <xacro:property name="J2_limit_upper"             value="${radians(143)}"/>
+  <xacro:property name="J2_limit_lower"             value="-1.5708"/>
+  <xacro:property name="J2_limit_upper"             value="1.5708"/>
   <xacro:property name="J2_limit_vel"               value="${pi}"/>
   <xacro:property name="J3_limit_effort"            value="0"/>
-  <xacro:property name="J3_limit_lower"             value="-1.4"/>
-  <xacro:property name="J3_limit_upper"             value="1.8"/>
+  <xacro:property name="J3_limit_lower"             value="0"/>
+  <xacro:property name="J3_limit_upper"             value="${pi}"/>
   <xacro:property name="J3_limit_vel"               value="${pi}"/>
   <xacro:property name="J4_limit_effort"            value="0"/>
@@ -19,6 +19,6 @@
   <xacro:property name="J4_limit_vel"               value="${pi}"/>
   <xacro:property name="J5_limit_effort"            value="0"/>
-  <xacro:property name="J5_limit_lower"             value="-0.75"/>
-  <xacro:property name="J5_limit_upper"             value="2.9"/>
+  <xacro:property name="J5_limit_lower"             value="0"/>
+  <xacro:property name="J5_limit_upper"             value="${pi}"/>
   <xacro:property name="J5_limit_vel"               value="${pi}"/>
   <xacro:property name="J6_limit_effort"            value="0"/>
@@ -178,5 +178,5 @@
     <origin
       xyz="0.0221 0 0"
-      rpy="1.5708 1.0391 1.5708" />
+      rpy="1.5708 1.5708 1.5708" />
     <parent
       link="$(arg robot_name)/J1" />
@@ -236,5 +236,5 @@
     <origin
       xyz="-0.06275 0.242 0"
-      rpy="-3.1416 0 1.8245" />
+      rpy="-3.1416 0 3.1416" />
     <parent
       link="$(arg robot_name)/J2" />
@@ -352,5 +352,5 @@
     <origin
       xyz="0 -0.012639 0.012639"
-      rpy="1.5708 0.80221 1.5708" />
+      rpy="1.5708 1.5708 1.5708" />
     <parent
       link="$(arg robot_name)/J4" />

Commit message: Updated joint limits for physical robots, added code in driver code writing commands to prevent gripper from overloading

File: hawaii_ros_ws/src/hawaii_descriptions/urdf/Student_Arm.urdf.xacro (robot description, xacro)
@@ -3,10 +3,10 @@
   <xacro:property name="robot_name"                 default="Student_Arm"/>
   <xacro:property name="J1_limit_effort"            value="0"/>
-  <xacro:property name="J1_limit_lower"             value="${-pi}"/>
-  <xacro:property name="J1_limit_upper"             value="${pi}"/>
+  <xacro:property name="J1_limit_lower"             value="${-pi/2}"/>
+  <xacro:property name="J1_limit_upper"             value="${pi/2}"/>
   <xacro:property name="J1_limit_vel"               value="${pi}"/>
   <xacro:property name="J2_limit_effort"            value="0"/>
   <xacro:property name="J2_limit_lower"             value="-1.5708"/>
-  <xacro:property name="J2_limit_upper"             value="1.5708"/>
+  <xacro:property name="J2_limit_upper"             value="1.1694"/>
   <xacro:property name="J2_limit_vel"               value="${pi}"/>
   <xacro:property name="J3_limit_effort"            value="0"/>

Commit message: changed arm to velocity profile type and got smooth teleop working

File: hawaii_ros_ws/src/hawaii_descriptions/urdf/Student_Arm.urdf.xacro (robot description, xacro)
@@ -11,6 +11,6 @@
   <xacro:property name="J2_limit_vel"               value="${pi}"/>
   <xacro:property name="J3_limit_effort"            value="0"/>
-  <xacro:property name="J3_limit_lower"             value="0"/>
-  <xacro:property name="J3_limit_upper"             value="${pi}"/>
+  <xacro:property name="J3_limit_lower"             value="0.08743"/>
+  <xacro:property name="J3_limit_upper"             value="3.05262"/>
   <xacro:property name="J3_limit_vel"               value="${pi}"/>
   <xacro:property name="J4_limit_effort"            value="0"/>
